File: driver_card_4234520/4234520.kicad_sch (KiCad schematic)
At the start: 39 parts, among them J1 Bus_ISA_8bit, J2 DC62_Female, U1 74LS74, U10 74LS155, U11 74LS02, U12 74LS09, U13 74LS244, U14 74LS244, U15 74LS21, U16 74LS244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

Commit message: change pin spacing on 62 pin connector and reconnect traces
Parts:
- J2: footprint Connector_Dsub:DSUB-62-HD_Female_Horizontal_P2.41x1.98mm_EdgePinOffset3.03mm_Housed_MountingHolesOffset4.94mm -> Connector_Dsub:DSUB-62-HD_Female_Horizontal_P2.41x2.54mm_EdgePinOffset9.40mm
Changed lines of the file:
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@@
       (effects (font (size 1.27 1.27)))
     )
-    (property "Footprint" "Connector_Dsub:DSUB-62-HD_Female_Horizontal_P2.41x1.98mm_EdgePinOffset3.03mm_Housed_MountingHolesOffset4.94mm" (at 257.81 85.09 0)
+    (property "Footprint" "Connector_Dsub:DSUB-62-HD_Female_Horizontal_P2.41x2.54mm_EdgePinOffset9.40mm" (at 257.81 85.09 0)
       (effects (font (size 1.27 1.27)) hide)
     )
